Commit message: 20260401_BG_urdfv4

File: δ1 & ε2/urdf/hylion_v4.urdf (robot description, URDF)
Before this commit: robot hylion, 31 links, 30 joints
Links:
- link base: geometry collision box size=0.15 0.14 0.23; visual mesh filename=../components/berkeley_humanoid_lite/mesh/base_visual.stl
- link soarm_left_wrist_link: geometry collision mesh filename=../components/so-arm/assets/sts3215_03a_no_horn_v1.stl; collision mesh filename=../components/so-arm/assets/wrist_roll_pitch_so101_v2.stl
- link soarm_right_wrist_link: geometry collision mesh filename=../components/so-arm/assets/sts3215_03a_no_horn_v1.stl; collision mesh filename=../components/so-arm/assets/wrist_roll_pitch_so101_v2.stl
Joints:
- joint soarm_left_base_joint: origin xyz=0 0.10 0.544 rpy=3.14159 0 0 -> xyz=0 0.12 0.82 rpy=3.14159 0 1.5708
- joint soarm_left_elbow_flex: limit lower=-1.69 upper=1.69 effort=10 velocity=10 -> lower=-1.6755 upper=1.6755 effort=10 velocity=10; origin xyz=-0.11257 -0.028 1.73763e-16 rpy=-3.63608e-16 8.74301e-16 1.5708 -> xyz=-0.11257 -0.028 1.73763e-16 rpy=-3.63608e-16 8.74301e-16 0
- joint soarm_left_gripper_frame_joint: axis (none) -> 0 0 0
- joint soarm_right_base_joint: origin xyz=0 -0.10 0.544 rpy=3.14159 0 0 -> xyz=0 -0.12 0.82 rpy=3.14159 0 -1.5708
- joint soarm_right_elbow_flex: limit lower=-1.69 upper=1.69 effort=10 velocity=10 -> lower=-1.6755 upper=1.6755 effort=10 velocity=10; origin xyz=-0.11257 -0.028 1.73763e-16 rpy=-3.63608e-16 8.74301e-16 1.5708 -> xyz=-0.11257 -0.028 1.73763e-16 rpy=-3.63608e-16 8.74301e-16 0
- joint soarm_right_gripper_frame_joint: axis (none) -> 0 0 0
